Commit message: change joint name

File: omni4_description/urdf/main.urdf.xacro (robot description, xacro)
@@ -36,37 +36,37 @@
 	</joint>
 	<xacro:rim_macro
-		name="left"
+		name="back_left"
 		color="0.3 0 0"
-		xyz="-0.04 0 0"
-		rpy="1.570796326794896 0 -1.570796326794896"/>
+		xyz="-0.03 0.03 0"
+		rpy="1.570796326794896 0 -2.35619449"/>
 	<xacro:rim_macro
-		name="back"
+		name="back_right"
 		color="0 0.3 0"
-		xyz="0 -0.04 0"
-		rpy="1.570796326794896 0 3.141592653589793"/>
+		xyz="-0.03 -0.03 0"
+		rpy="1.570796326794896 0 -0.7853981634"/>
 	<xacro:rim_macro
-		name="right"
+		name="front_right"
 		color="0 0 0.3"
-		xyz="0.04 0 0"
-		rpy="1.570796326794896 0 1.570796326794896"/>
+		xyz="0.03 -0.03 0"
+		rpy="1.570796326794896 0 0.7853981634"/>
 	<xacro:rim_macro
-		name="front"
+		name="front_left"
 		color="0 0.3 0.3"
-		xyz="0 0.04 0"
-		rpy="1.570796326794896 0 0"/>
+		xyz="0.03 0.03 0"
+		rpy="1.570796326794896 0 2.35619449"/>
 	<gazebo reference="base_link">
     		<material>Gazebo/White</material>
   	</gazebo>
-	<gazebo reference="rim_left_link">
+	<gazebo reference="rim_back_left_link">
     		<material>Gazebo/Red</material>
   	</gazebo>
-	<gazebo reference="rim_back_link">
+	<gazebo reference="rim_back_right_link">
     		<material>Gazebo/Green</material>
   	</gazebo>
-	<gazebo reference="rim_right_link">
+	<gazebo reference="rim_front_right_link">
     		<material>Gazebo/Blue</material>
   	</gazebo>
-	<gazebo reference="rim_front_link">
-    		<material>Gazebo/Black</material>
+	<gazebo reference="rim_front_left_link">
+    		<material>Gazebo/SkyBlue</material>
   	</gazebo>
 	<gazebo>

Commit message: add lidar,imu

File: omni4_description/urdf/main.urdf.xacro (robot description, xacro)
@@ -34,4 +34,31 @@
 		<child link="base_link" />
 		<origin xyz="0 0 0.01905" rpy="0 0 0"/>
+	</joint>
+	<link name="lidar_link">
+		<visual>
+			<geometry>
+				<mesh filename="package://omni4_description/mesh/hokuyo.dae" scale="0.5 0.5 0.5"/>
+			</geometry>
+			<material name="LightGrey">
+				<color rgba="0.7 0.7 0.7 1.0"/>
+			</material>
+		</visual>
+		<collision>
+			<geometry>
+				<mesh filename="package://omni4_description/mesh/hokuyo.dae" scale="0.5 0.5 0.5"/>
+			</geometry>
+		</collision>
+	</link>
+	<joint name="lidar_joint" type="fixed">
+		<parent link="base_link"/>
+		<child link="lidar_link"/>
+		<origin xyz="0 0 0.01" rpy="0 0 0"/>
+	</joint>
+	<link name="imu_link">
+	</link>
+	<joint name="imu_joint" type="fixed">
+		<parent link="base_link"/>
+		<child link="imu_link"/>
+		<origin xyz="0 0 0" rpy="0 0 0"/>
 	</joint>
 	<xacro:rim_macro
@@ -75,3 +102,52 @@
 		</plugin>
 	</gazebo>
+	  <!--LIDAR-->
+	<gazebo reference="lidar_link">
+	<material>Gazebo/Black</material>
+	<turnGravityOff>false</turnGravityOff>
+	<sensor type="ray" name="head_hokuyo_sensor">
+		<pose>$0 0 0 0 0 0</pose>
+		<visualize>true</visualize>
+		<update_rate>40</update_rate>
+		<ray>
+		<scan>
+			<horizontal>
+			<samples>720</samples>
+			<resolution>1</resolution>
+			<min_angle>-3.1415</min_angle>
+			<max_angle>3.1415</max_angle>
+			</horizontal>
+		</scan>
+		<range>
+			<min>0.10</min>
+			<max>5.0</max>
+			<resolution>0.001</resolution>
+		</range>
+		</ray>
+		<plugin name="gazebo_ros_head_hokuyo_controller" filename="libgazebo_ros_laser.so">
+		<topicName>/scan</topicName>
+		<frameName>lidar_link</frameName>
+		</plugin>
+	</sensor>
+	</gazebo>
+	<gazebo reference="imu_link">
+		<gravity>true</gravity>
+		<sensor name="imu_sensor" type="imu">
+		<always_on>true</always_on>
+		<update_rate>100</update_rate>
+		<visualize>true</visualize>
+		<topic>__default_topic__</topic>
+		<plugin filename="libgazebo_ros_imu_sensor.so" name="imu_plugin">
+			<topicName>imu_data</topicName>
+			<bodyName>imu_link</bodyName>
+			<updateRateHZ>10.0</updateRateHZ>
+			<gaussianNoise>0.0</gaussianNoise>
+			<xyzOffset>0 0 0</xyzOffset>
+			<rpyOffset>0 0 0</rpyOffset>
+			<frameName>imu_link</frameName>
+			<initialOrientationAsReference>false</initialOrientationAsReference>
+		</plugin>
+		<pose>0 0 0 0 0 0</pose>
+		</sensor>
+	</gazebo>
 </robot>

Commit message: fix kinematic

File: omni4_description/urdf/main.urdf.xacro (robot description, xacro)
@@ -63,37 +63,37 @@
 	</joint>
 	<xacro:rim_macro
-		name="back_left"
+		name="front_left"
 		color="0.3 0 0"
 		xyz="-0.03 0.03 0"
+		rpy="1.570796326794896 0 0.7853981634"/>
+	<xacro:rim_macro
+		name="back_left"
+		color="0 0.3 0"
+		xyz="-0.03 -0.03 0"
+		rpy="1.570796326794896 0 2.35619449"/>
+	<xacro:rim_macro
+		name="back_right"
+		color="0 0 0.3"
+		xyz="0.03 -0.03 0"
 		rpy="1.570796326794896 0 -2.35619449"/>
 	<xacro:rim_macro
-		name="back_right"
-		color="0 0.3 0"
-		xyz="-0.03 -0.03 0"
-		rpy="1.570796326794896 0 -0.7853981634"/>
-	<xacro:rim_macro
 		name="front_right"
-		color="0 0 0.3"
-		xyz="0.03 -0.03 0"
-		rpy="1.570796326794896 0 0.7853981634"/>
-	<xacro:rim_macro
-		name="front_left"
 		color="0 0.3 0.3"
 		xyz="0.03 0.03 0"
-		rpy="1.570796326794896 0 2.35619449"/>
+		rpy="1.570796326794896 0 -0.7853981634"/>
 	<gazebo reference="base_link">
     		<material>Gazebo/White</material>
   	</gazebo>
-	<gazebo reference="rim_back_left_link">
+	<gazebo reference="rim_front_right_link">
     		<material>Gazebo/Red</material>
   	</gazebo>
-	<gazebo reference="rim_back_right_link">
+	<gazebo reference="rim_front_left_link">
     		<material>Gazebo/Green</material>
   	</gazebo>
-	<gazebo reference="rim_front_right_link">
+	<gazebo reference="rim_back_left_link">
     		<material>Gazebo/Blue</material>
   	</gazebo>
-	<gazebo reference="rim_front_left_link">
-    		<material>Gazebo/SkyBlue</material>
+	<gazebo reference="rim_back_right_link">
+    		<material>Gazebo/Yellow</material>
   	</gazebo>
 	<gazebo>

Commit message: gmapping

File: omni4_description/urdf/main.urdf.xacro (robot description, xacro)
@@ -5,12 +5,12 @@
 	<link name="base_link">
 	<inertial>
-		<mass value="0.07862944645"/>
+		<mass value="0.15726"/>
 		<inertia
-			ixx="0.00002035985530754"
+			ixx="0.00004718"
 			ixy="0"
 			ixz="0"
-			iyy="0.00002035985530754"
+			iyy="0.00004718"
 			iyz="0"
-			izz="0.00003945961663220"/>
+			izz="0.000083876"/>
 		</inertial>
 	<visual>
@@ -53,5 +53,5 @@
 		<parent link="base_link"/>
 		<child link="lidar_link"/>
-		<origin xyz="0 0 0.01" rpy="0 0 0"/>
+		<origin xyz="0 0 0.02" rpy="0 0 0"/>
 	</joint>
 	<link name="imu_link">
@@ -108,5 +108,5 @@
 	<sensor type="ray" name="head_hokuyo_sensor">
 		<pose>$0 0 0 0 0 0</pose>
-		<visualize>true</visualize>
+		<visualize>false</visualize>
 		<update_rate>40</update_rate>
 		<ray>

File: omni4_description/urdf/roller.urdf.xacro (robot description, xacro)
@@ -31,4 +31,6 @@
 	<gazebo reference="roller_${name}_rim_${parent}_link">
     		<material>Gazebo/Black</material>
+			<mu value="1"/>
+			<mu2 value="1"/>
   	</gazebo>
 		<joint name="roller_${name}_rim_${parent}_joint" type="continuous">
